Commit message: Correct URDF foot and leg, also add contact sensor API in the USD

File: exts/MicroSpot_implementation/assets/URDF/spotmicroaiean.urdf (robot description, URDF)
Before this commit: robot SpotMicroAI, 19 links, 18 joints
Links:
- removed link base_link
- removed link front_left_leg_link
- removed link front_left_toe_link
- removed link front_right_leg_link
- removed link front_right_toe_link
- removed link rear_left_leg_link
- removed link rear_left_toe_link
- removed link rear_right_leg_link
- removed link rear_right_toe_link
- added link base, mass 0.94447; collision box size=0.2 0.11 0.07; visual mesh filename=meshes/stl_ean/STL/Base.STL scale=0.001 0.001 0.001
- added link front_left_toe_link_FOOT, mass 0.0; collision sphere radius=0.02; visual mesh filename=meshes/stl_ean/STL/Foot_Tip.STL scale=0.001 0.001 0.001
- added link front_left_toe_link_THIGH, mass 0.1942; collision box size=0.028 0.036 0.12; visual mesh filename=meshes/stl_ean/STL/left_arm.STL scale=0.001 0.001 0.001
- added link front_right_toe_link_FOOT, mass 0.0; collision sphere radius=0.02; visual mesh filename=meshes/stl_ean/STL/Foot_Tip.STL scale=0.001 0.001 0.001
- added link front_right_toe_link_THIGH, mass 0.19412; collision box size=0.028 0.036 0.12; visual mesh filename=meshes/stl_ean/STL/right_arm.STL scale=0.001 0.001 0.001
- added link rear_left_toe_link_FOOT, mass 0.0; collision sphere radius=0.02; visual mesh filename=meshes/stl_ean/STL/Foot_Tip.STL scale=0.001 0.001 0.001
- added link rear_left_toe_link_THIGH, mass 0.1942; collision box size=0.028 0.036 0.12; visual mesh filename=meshes/stl_ean/STL/left_arm.STL scale=0.001 0.001 0.001
- added link rear_right_toe_link_FOOT, mass 0.0; collision sphere radius=0.02; visual mesh filename=meshes/stl_ean/STL/Foot_Tip.STL scale=0.001 0.001 0.001
- added link rear_right_toe_link_THIGH, mass 0.19412; collision box size=0.028 0.036 0.12; visual mesh filename=meshes/stl_ean/STL/right_arm.STL scale=0.001 0.001 0.001
Joints:
- joint base_front: parent base_link -> base
- joint base_rear: parent base_link -> base
- joint joint_front_left_foot: parent front_left_leg_link -> front_left_toe_link_THIGH
- joint joint_front_left_leg: child front_left_leg_link -> front_left_toe_link_THIGH
- joint joint_front_left_shoulder: parent base_link -> base
- joint joint_front_left_toe: child front_left_toe_link -> front_left_toe_link_FOOT
- joint joint_front_right_foot: parent front_right_leg_link -> front_right_toe_link_THIGH
- joint joint_front_right_leg: child front_right_leg_link -> front_right_toe_link_THIGH
- joint joint_front_right_shoulder: parent base_link -> base
- joint joint_front_right_toe: child front_right_toe_link -> front_right_toe_link_FOOT
- joint joint_rear_left_foot: parent rear_left_leg_link -> rear_left_toe_link_THIGH
- joint joint_rear_left_leg: child rear_left_leg_link -> rear_left_toe_link_THIGH
- joint joint_rear_left_shoulder: parent base_link -> base
- joint joint_rear_left_toe: child rear_left_toe_link -> rear_left_toe_link_FOOT
- joint joint_rear_right_foot: parent rear_right_leg_link -> rear_right_toe_link_THIGH
- joint joint_rear_right_leg: child rear_right_leg_link -> rear_right_toe_link_THIGH
- joint joint_rear_right_shoulder: parent base_link -> base
- joint joint_rear_right_toe: child rear_right_toe_link -> rear_right_toe_link_FOOT

Commit message: solving dumb erros, URDF stop using package routes and remove the disable contact_forces line

File: exts/MicroSpot_implementation/assets/URDF/spotmicroaiean.urdf (robot description, URDF)
Before this commit: robot SpotMicroAI, 19 links, 18 joints
Links:
- removed link front_left_toe_link_THIGH
- removed link front_right_toe_link_THIGH
- removed link rear_left_toe_link_THIGH
- removed link rear_right_toe_link_THIGH
- added link front_left_leg_link_THIGH, mass 0.1942; collision box size=0.028 0.036 0.12; visual mesh filename=meshes/stl_ean/STL/left_arm.STL scale=0.001 0.001 0.001
- added link front_right_leg_link_THIGH, mass 0.19412; collision box size=0.028 0.036 0.12; visual mesh filename=meshes/stl_ean/STL/right_arm.STL scale=0.001 0.001 0.001
- added link rear_left_leg_link_THIGH, mass 0.1942; collision box size=0.028 0.036 0.12; visual mesh filename=meshes/stl_ean/STL/left_arm.STL scale=0.001 0.001 0.001
- added link rear_right_leg_link_THIGH, mass 0.19412; collision box size=0.028 0.036 0.12; visual mesh filename=meshes/stl_ean/STL/right_arm.STL scale=0.001 0.001 0.001
Joints:
- joint joint_front_left_foot: parent front_left_toe_link_THIGH -> front_left_leg_link_THIGH
- joint joint_front_left_leg: child front_left_toe_link_THIGH -> front_left_leg_link_THIGH
- joint joint_front_right_foot: parent front_right_toe_link_THIGH -> front_right_leg_link_THIGH
- joint joint_front_right_leg: child front_right_toe_link_THIGH -> front_right_leg_link_THIGH
- joint joint_rear_left_foot: parent rear_left_toe_link_THIGH -> rear_left_leg_link_THIGH
- joint joint_rear_left_leg: child rear_left_toe_link_THIGH -> rear_left_leg_link_THIGH
- joint joint_rear_right_foot: parent rear_right_toe_link_THIGH -> rear_right_leg_link_THIGH
- joint joint_rear_right_leg: child rear_right_toe_link_THIGH -> rear_right_leg_link_THIGH
